Commit message: it flies straight up

File: urdf/m100_no_frills_backup.xacro (robot description, xacro)
@@ -2,5 +2,4 @@
 <robot name="m100_barebones" xmlns:xacro="http://www.ros.org/wiki/xacro">
   <xacro:arg name="robot_namespace" default="/" />
-  <xacro:property name="clean_ns" value="${'$(arg robot_namespace)'.strip('/')}" />
   <link name="base_footprint"/>
   <joint name="base_joint" type="fixed">
@@ -35,5 +34,5 @@
       <updateRate>100.0</updateRate>
       <bodyName>base_link</bodyName>
-      <base_link_frame>${clean_ns}/base_link</base_link_frame>
+      <base_link_frame>$(arg robot_namespace)/base_link</base_link_frame>
       <topicName>cmd_vel</topicName>
       <stateTopic>ground_truth/state</stateTopic>
@@ -63,5 +62,5 @@
       <updateRate>100.0</updateRate>
       <bodyName>base_link</bodyName>
-      <frameId>${clean_ns}/base_link</frameId>
+      <frameId>$(arg robot_namespace)/base_link</frameId>
       <topicName>raw_imu</topicName>
     </plugin>
